Commit message: 加入巡线脚本

File: racecar_description/urdf/racecar.xacro (robot description, xacro)
@@ -192,5 +192,5 @@
   </link>
   <joint name="zed_camera_joint" type="fixed">
-    <origin xyz="0.390 0 0.04" rpy="0 0 0"/>
+    <origin xyz="0.390 0 0.1" rpy="0 0.2 0"/>
     <parent link="chassis"/>
     <child link="zed_camera_link"/>

Commit message: 修复建图bug，写四轮摄像头博客的时候把激光雷达关了，干了件蠢事导致大家建不了图

File: racecar_description/urdf/racecar.xacro (robot description, xacro)
@@ -192,5 +192,5 @@
   </link>
   <joint name="zed_camera_joint" type="fixed">
-    <origin xyz="0.390 0 0.1" rpy="0 0.2 0"/>
+    <origin xyz="0.390 0 0" rpy="0 0 0"/>
     <parent link="chassis"/>
     <child link="zed_camera_link"/>

Commit message: 修改readme增加control报警告导致车不走解决办法

File: racecar_description/urdf/racecar.xacro (robot description, xacro)
@@ -192,5 +192,5 @@
   </link>
   <joint name="zed_camera_joint" type="fixed">
-    <origin xyz="0.390 0 0" rpy="0 0 0"/>
+    <origin xyz="0.390 0 0.2" rpy="0 0 0"/>
     <parent link="chassis"/>
     <child link="zed_camera_link"/>

Commit message: 修改模型试用红绿灯检测

File: racecar_description/urdf/racecar.xacro (robot description, xacro)
@@ -192,5 +192,5 @@
   </link>
   <joint name="zed_camera_joint" type="fixed">
-    <origin xyz="0.390 0 0.2" rpy="0 0 0"/>
+    <origin xyz="0.390 0 0.2" rpy="0 0.2 0"/>
     <parent link="chassis"/>
     <child link="zed_camera_link"/>
